File: MEGA_MSX/MEGA_MSX.sch (EAGLE design)
At the start: 8 parts, among them IC1 TINY85

Commit message: Cleanup and organization of some directories
Parts:
- removed C1: 100nf, rcl:C-EU050-024X044
- removed C2: 10nf, rcl:C-EU050-024X044
- removed R2: 10K, Pontentiometer:3RP/1610NTHRU
- removed R3: 1k, rcl:R-EU_0204/7
- removed S1: (no value), switch-omron:40-XX
- removed SV1: (no value), con-lstb:MA09-1
- added C3: 100n, rcl:C-EUC0805
- added X1: MEGA-1, con-subd:M09DS
- added X2: MEGA-2, con-subd:M09DS
- added X3: MSX, con-molex:22-23-2091
- IC1: value TINY85 -> ATMegaxx8; device atmel:TINY15LP -> atmel:MEGA8-AI
- R1: value 1k -> 10k; device rcl:R-EU_0204/7 -> rcl:R-EU_R0805
Connections:
- removed net +5V: C1.1, IC1.VCC, R1.2, R2.E, R3.2, SV1.5
- removed net BUTTON: IC1.(ADC2)PB3, S1.P1
- removed net DOWN: IC1.(OCP)PB1, R3.1, SV1.2
- removed net POT: C2.1, IC1.(ADC0)PB5, R2.S
- removed net PULSE: IC1.(ADC1)PB2, SV1.8
- removed net TRG-A: IC1.(ADC3)PB4, SV1.6
- removed net UP: IC1.(AREF)PB0, R1.1, SV1.1
- new net !RESET: IC1.PC6(/RESET), R1.1
- new net MEGA1_BTA_BTB: IC1.PB0(ICP), X1-6.M
- new net MEGA1_DOWN: IC1.PB2(SS/OC1B), X1-2.M
- new net MEGA1_LEFT: IC1.PB3(MOSI/OC2), X1-3.M
- new net MEGA1_RIGHT: IC1.PB4(MISO), X1-4.M
- new net MEGA1_SELECT: IC1.PB7(XTAL2/TOSC2), X1-7.M
- new net MEGA1_START_BTC: IC1.PB5(SCK), X1-9.M
- new net MEGA1_UP: IC1.PB1(OC1A), X1-1.M
- new net MEGA2_BTA_BTB: IC1.PC1(ADC1), X2-6.M
- new net MEGA2_DOWN: IC1.PC2(ADC2), X2-2.M
- new net MEGA2_LEFT: IC1.PC3(ADC3), X2-3.M
- new net MEGA2_RIGHT: IC1.PC4(ADC4/SDA), X2-4.M
- new net MEGA2_SELECT: IC1.PB6(XTAL1/TOSC1), X2-7.M
- new net MEGA2_START_BTC: IC1.PC5(ADC5/SCL), X2-9.M
- new net MEGA2_UP: IC1.PC0(ADC0), X2-1.M
- new net MEX_RIGHT: IC1.PD3(INT1), X3-4.S
- new net MSX_DOWN: IC1.PD1(TXD), X3-2.S
- new net MSX_LEFT: IC1.PD2(INT0), X3-3.S
- new net MSX_PULSE: IC1.PD7(AIN1), X3-8.S
- new net MSX_TRGA: IC1.PD5(T1), X3-6.S
- new net MSX_TRGB: IC1.PD6(AIN0), X3-7.S
- new net MSX_UP: IC1.PD0(RXD), X3-1.S
- new net VCC: C3.1, IC1.AREF, IC1.AVCC, IC1.VCC@1, IC1.VCC@2, R1.2, X1-5.M, X2-5.M, X3-5.S
- net GND: now also C3.2, IC1.GND@1, IC1.GND@2, X1-8.M, X2-8.M, X3-9.S; no longer C1.2, C2.2, R2.A, S1.S, S1.S1, SV1.9
Other:
- note added: "Dual Megadrive controller adapter for MSX"
- moved on the sheet: R1
