File: Paddle_Revisited/Discrete/circuit/Vaus Arkanoid paddle.brd (EAGLE design)
At the start: 84 x 37 mm, 23 parts, among them IC1 4040N, IC2 74165N, IC3 74LS00N, IC4 LM556N

Commit message: Cleanup and organization of some directories
Parts:
- added C9: 100nf, rcl:C050-024X044
- C2: value 15n -> 10n
- R3: value 1k -> 1k5
- moved R1 26.2 mm to (71.1, 14.0), turned to 0 degrees
- moved R4 5.99 mm to (71.1, 11.4)
- moved C4 3.17 mm to (59.1, 36.2)
- moved C10 1.90 mm to (62.9, 40.0)
- moved R7 1.27 mm to (69.8, 39.4)
Connections:
- net DOUT: now also C9.1
- net GND: now also C9.2
- net N$15: now also R5.1; no longer R5.3
- net N$22: now also R5.3; no longer R5.1
Routing:
- net GND: track 168.4 -> 147.4 mm
- net N$15: track 25.0 -> 40.2 mm
- net N$1: track 113.7 -> 121.6 mm
- net N$13: track 20.8 -> 28.0 mm
- net N$12: track 63.4 -> 69.7 mm
- net VCC: track 246.1 -> 252.2 mm
- net N$22: track 63.3 -> 58.0 mm
- net DOUT: track 31.4 -> 33.0 mm
- net PULSE: track 55.6 -> 54.9 mm
Other:
- board text added: "Danjovic 2019"
- board text added: "Vaus Arkanoid Paddle"
- board text added: "Vaus Arkanopid Paddle"
- board text removed: "Danjovic 2018"
- board text removed: "Taito Arkanoid Paddle"
- board text removed: "Taito Arkanopid Paddle"

Commit message: Updated component values
Parts:
- C5: value 1k -> 100nf
Changed lines of the file:
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@@
 <layers>
 <layer number="1" name="Top" color="4" fill="1" visible="no" active="yes"/>
-<layer number="16" name="Bottom" color="1" fill="1" visible="yes" active="yes"/>
+<layer number="16" name="Bottom" color="1" fill="1" visible="no" active="yes"/>
 <layer number="17" name="Pads" color="2" fill="1" visible="yes" active="yes"/>
 <layer number="18" name="Vias" color="2" fill="1" visible="yes" active="yes"/>
@@
 <attribute name="VALUE" x="61.214" y="34.036" size="1.27" layer="27" ratio="10"/>
 </element>
-<element name="C5" library="rcl" package="C050-024X044" value="1k" x="55.245" y="38.1" smashed="yes" rot="R270">
+<element name="C5" library="rcl" package="C050-024X044" value="100nf" x="55.245" y="38.1" smashed="yes" rot="R270">
 <attribute name="NAME" x="53.721" y="41.402" size="1.27" layer="25" ratio="10"/>
 <attribute name="VALUE" x="52.451" y="32.893" size="1.27" layer="27" ratio="10"/>
