File: EXPS2/circuit/external/EXPS2.brd (EAGLE design)
At the start: 59.1 x 59.1 mm, 13 parts, among them IC1 ATMEGA-8P, Q1 16MHz

Commit message: Updated Single Sided Board
Parts:
- added ISP: (no value), con-harting-ml:ML6
- added Q2: 16MHz, crystal:TC26H
- K2: device con-yamaichi:MDIN06SS -> con-yamaichi:MDIN06S
- R1, R2, R3: device rcl:0204/5 -> rcl:0204/7
- moved C1 2.54 mm to (38.1, 26.7)
- moved IC1 2.54 mm to (27.9, 30.5)
- moved Q1 2.54 mm to (38.1, 35.6)
- moved C4 1.27 mm to (19.1, 30.5)
Connections:
- net !RESET: now also ISP.5
- net GND: now also ISP.6
- net MISO: now also ISP.1
- net MOSI: now also ISP.4
- net SCK: now also ISP.3
- net VCC: now also ISP.2
- net XTAL1: now also Q2.2
- net XTAL2: now also Q2.1
Routing:
- net GND: track 262.1 -> 223.4 mm, vias 0 -> 2
- net !RESET: track 83.2 -> 121.7 mm, vias 0 -> 2
- net VCC: track 111.9 -> 144.2 mm, vias 2 -> 4
- net MOSI: track 0.00 -> 30.3 mm
- net SCK: track 0.00 -> 28.9 mm
- net MISO: track 0.00 -> 24.6 mm
- net CLK: track 68.0 -> 88.9 mm
- net DAT: track 77.2 -> 94.5 mm
- net SEL_D: track 38.1 -> 31.0 mm
- net COL_2: track 45.0 -> 40.2 mm
- net COL_4: track 50.3 -> 46.2 mm
- net COL_0: track 38.4 -> 35.3 mm
- net SEL_B: track 21.0 -> 18.5 mm
- net COL_3: track 55.1 -> 52.5 mm
- net XTAL2: track 13.1 -> 15.6 mm
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Other:
- board text added: "2021"
- board text added: "Danjovic"
- board text added: "JLCJLCJLCJLC"
