File: EXPS2/circuit/external/EXPS2.sch (EAGLE design)
At the start: 12 parts, among them IC1 ATMEGA-8P, Q1 16MHz

Commit message: Updated Single Sided Board
Parts:
- added ISP: (no value), con-harting-ml:ML6
- added Q2: 16MHz, crystal:CRYSTALTC26H
- K2: device con-yamaichi:MD06SS -> con-yamaichi:MD06S
- R1, R2, R3: device rcl:R-EU_0204/5 -> rcl:R-EU_0204/7
Connections:
- net !RESET: now also ISP.5
- net GND: now also ISP.6
- net MISO: now also ISP.1
- net MOSI: now also ISP.4
- net SCK: now also ISP.3
- net VCC: now also ISP.2
- net XTAL1: now also Q2.2
- net XTAL2: now also Q2.1
Other:
- note added: "Alternative"
Changed lines of the file:
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@@
 <part name="P+1" library="supply1" deviceset="VCC" device=""/>
 <part name="P+2" library="supply1" deviceset="VCC" device=""/>
-<part name="R1" library="rcl" deviceset="R-EU_" device="0204/5" value="10k"/>
-<part name="R2" library="rcl" deviceset="R-EU_" device="0204/5" value="10k"/>
+<part name="R1" library="rcl" deviceset="R-EU_" device="0204/7" value="10k"/>
+<part name="R2" library="rcl" deviceset="R-EU_" device="0204/7" value="10k"/>
 <part name="FRAME1" library="frames" deviceset="A4L-LOC" device=""/>
-<part name="K2" library="con-yamaichi" deviceset="MD06SS" device=""/>
 <part name="K3" library="con-berg" deviceset="PN87520" device=""/>
 <part name="C2" library="rcl" deviceset="C-EU" device="050-024X044" value="22p"/>
@@
 <part name="C3" library="rcl" deviceset="C-EU" device="050-024X044" value="22p"/>
 <part name="Q1" library="crystal" deviceset="CRYSTAL" device="HC49U-V" value="16MHz"/>
-<part name="R3" library="rcl" deviceset="R-EU_" device="0204/5" value="10k"/>
+<part name="R3" library="rcl" deviceset="R-EU_" device="0204/7" value="10k"/>
 <part name="P+4" library="supply1" deviceset="VCC" device=""/>
 <part name="P+5" library="supply1" deviceset="VCC" device=""/>
@@
 <part name="GND2" library="supply1" deviceset="GND" device=""/>
 <part name="C4" library="rcl" deviceset="CPOL-EU" device="E2.5-6" value="220u"/>
+<part name="K2" library="con-yamaichi" deviceset="MD06S" device=""/>
+<part name="ISP" library="con-harting-ml" deviceset="ML6" device=""/>
+<part name="P+8" library="supply1" deviceset="VCC" device=""/>
+<part name="GND7" library="supply1" deviceset="GND" device=""/>
+<part name="Q2" library="crystal" deviceset="CRYSTAL" device="TC26H" value="16MHz"/>
 </parts>
 <sheets>
@@
 <wire x1="226.314" y1="102.87" x2="226.314" y2="26.67" width="0.1524" layer="94"/>
 <wire x1="236.474" y1="102.87" x2="236.474" y2="26.67" width="0.1524" layer="94"/>
+<wire x1="226.06" y1="162.56" x2="248.92" y2="162.56" width="0.1524" layer="94" style="shortdash"/>
+<wire x1="248.92" y1="162.56" x2="248.92" y2="147.32" width="0.1524" layer="94" style="shortdash"/>
+<wire x1="248.92" y1="147.32" x2="226.06" y2="147.32" width="0.1524" layer="94" style="shortdash"/>
+<wire x1="226.06" y1="147.32" x2="226.06" y2="162.56" width="0.1524" layer="94" style="shortdash"/>
+<text x="226.822" y="148.082" size="1.27" layer="94">Alternative</text>
 </plain>
 <instances>
@@
 </instance>
 <instance part="FRAME1" gate="G$1" x="0" y="0"/>
-<instance part="K2" gate="G$1" x="68.58" y="50.8" rot="R180"/>
 <instance part="K3" gate="G$1" x="66.04" y="86.36" rot="MR0"/>
 <instance part="C2" gate="G$1" x="193.04" y="121.92"/>
@@
 <instance part="GND2" gate="1" x="45.72" y="109.22" rot="MR0"/>
 <instance part="C4" gate="G$1" x="223.52" y="121.92"/>
+<instance part="K2" gate="G$1" x="68.58" y="50.8" rot="R180"/>
+<instance part="ISP" gate="1" x="137.16" y="71.12" rot="R180"/>
+<instance part="P+8" gate="VCC" x="147.32" y="73.66" smashed="yes" rot="MR90">
+<attribute name="VALUE" x="152.4" y="73.66" size="1.778" layer="96" rot="MR0"/>
+</instance>
+<instance part="GND7" gate="1" x="144.78" y="66.04" rot="MR0"/>
+<instance part="Q2" gate="G$1" x="236.22" y="154.94" smashed="yes" rot="R90">
+<attribute name="NAME" x="233.68" y="156.464" size="1.778" layer="95" rot="R180"/>
+<attribute name="VALUE" x="238.76" y="154.94" size="1.778" layer="96"/>
+</instance>
 </instances>
 <busses>
@@
 </segment>
 <segment>
-<pinref part="K2" gate="G$1" pin="3"/>
 <pinref part="GND5" gate="1" pin="GND"/>
 <wire x1="78.74" y1="48.26" x2="83.82" y2="48.26" width="0.1524" layer="91"/>
 <wire x1="83.82" y1="48.26" x2="83.82" y2="40.64" width="0.1524" layer="91"/>
+<pinref part="K2" gate="G$1" pin="3"/>
 </segment>
 <segment>
@@
 <wire x1="45.72" y1="116.84" x2="45.72" y2="111.76" width="0.1524" layer="91"/>
 <pinref part="GND2" gate="1" pin="GND"/>
+</segment>
+<segment>
+<pinref part="ISP" gate="1" pin="6"/>
+<pinref part="GND7" gate="1" pin="GND"/>
 </segment>
 </net>
@@
 </segment>
 <segment>
-<pinref part="K2" gate="G$1" pin="4"/>
 <pinref part="P+5" gate="VCC" pin="VCC"/>
 <wire x1="88.9" y1="50.8" x2="78.74" y2="50.8" width="0.1524" layer="91"/>
+<pinref part="K2" gate="G$1" pin="4"/>
 </segment>
 <segment>
@@
 <pinref part="P+6" gate="VCC" pin="VCC"/>
 <wire x1="45.72" y1="119.38" x2="38.1" y2="119.38" width="0.1524" layer="91"/>
+</segment>
+<segment>
+<pinref part="ISP" gate="1" pin="2"/>
+<pinref part="P+8" gate="VCC" pin="VCC"/>
 </segment>
 </net>
@@
 <wire x1="101.6" y1="86.36" x2="101.6" y2="53.34" width="0.1524" layer="91"/>
 <pinref part="K3" gate="G$1" pin="3"/>
-<pinref part="K2" gate="G$1" pin="5"/>
 <wire x1="78.74" y1="53.34" x2="109.22" y2="53.34" width="0.1524" layer="91"/>
 <junction x="101.6" y="53.34"/>
 <wire x1="68.58" y1="86.36" x2="101.6" y2="86.36" width="0.1524" layer="91"/>
 <junction x="101.6" y="86.36"/>
+<pinref part="K2" gate="G$1" pin="5"/>
 </segment>
 </net>
@@
 <pinref part="R2" gate="G$1" pin="1"/>
 <pinref part="IC1" gate="G$1" pin="PB1(OC1A)"/>
-<pinref part="K2" gate="G$1" pin="1"/>
 <wire x1="104.14" y1="88.9" x2="104.14" y2="43.18" width="0.1524" layer="91"/>
 <wire x1="104.14" y1="43.18" x2="78.74" y2="43.18" width="0.1524" layer="91"/>
@@
 <wire x1="68.58" y1="88.9" x2="104.14" y2="88.9" width="0.1524" layer="91"/>
 <junction x="104.14" y="88.9"/>
+<pinref part="K2" gate="G$1" pin="1"/>
 </segment>
 </net>
@@
 <junction x="185.42" y="129.54"/>
 </segment>
+<segment>
+<wire x1="236.22" y1="160.02" x2="236.22" y2="157.48" width="0.1524" layer="91"/>
+<pinref part="Q2" gate="G$1" pin="2"/>
+</segment>
 </net>
 <net name="XTAL2" class="0">
@@
 <junction x="185.42" y="124.46"/>
 </segment>
+<segment>
+<wire x1="236.22" y1="149.86" x2="236.22" y2="152.4" width="0.1524" layer="91"/>
+<pinref part="Q2" gate="G$1" pin="1"/>
+</segment>
 </net>
 <net name="!RESET" class="0">
@@
 <pinref part="IC1" gate="G$1" pin="PC6(/RESET)"/>
 <pinref part="R3" gate="G$1" pin="2"/>
+<label x="172.72" y="147.32" size="1.778" layer="95"/>
+</segment>
+<segment>
+<wire x1="119.38" y1="68.58" x2="129.54" y2="68.58" width="0.1524" layer="91"/>
+<pinref part="ISP" gate="1" pin="5"/>
+<label x="121.92" y="68.58" size="1.778" layer="95"/>
 </segment>
 </net>
@@
 <label x="111.76" y="91.44" size="1.778" layer="95"/>
 </segment>
+<segment>
+<wire x1="119.38" y1="73.66" x2="129.54" y2="73.66" width="0.1524" layer="91"/>
+<pinref part="ISP" gate="1" pin="1"/>
+<label x="121.92" y="73.66" size="1.778" layer="95"/>
+</segment>
 </net>
 <net name="SCK" class="0">
@@
 <label x="111.76" y="88.9" size="1.778" layer="95"/>
 </segment>
+<segment>
+<wire x1="119.38" y1="71.12" x2="129.54" y2="71.12" width="0.1524" layer="91"/>
+<pinref part="ISP" gate="1" pin="3"/>
+<label x="121.92" y="71.12" size="1.778" layer="95"/>
+</segment>
 </net>
 <net name="MOSI" class="0">
@@
 <label x="111.76" y="93.98" size="1.778" layer="95"/>
 </segment>
-</net>
+<segment>
+<wire x1="154.94" y1="71.12" x2="144.78" y2="71.12" width="0.1524" layer="91"/>
+<pinref part="ISP" gate="1" pin="4"/>
+<label x="147.32" y="71.12" size="1.778" layer="95"/>
+</segment>
+</net>
