File: FA-32/C3427-3.sch (EAGLE design)
At the start: 50 parts, among them IC1 LA6358N, J1 PJ-301, J2 PJ-301, J3 PJ-201, K1 FBR211, K1(*) 351, T1 2SC945, T1(*) BC338

Commit message: Update board, added images
Parts:
- added J12(*): PJ-325, AudioJack:PJ-325
- renumbered K2 to J4
Connections:
- net EAR: now also J12(*).5
- net GND: now also J1.C, J12(*).1, J12(*).2, J12(*).4, J2.C
- net MIC: now also J12(*).3
Other:
- moved on the sheet: K1(*), T1(*)
Changed lines of the file:
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@@
 <part name="J2" library="Jack-PJ" deviceset="PJ-" device="301"/>
 <part name="J3" library="Jack-PJ" deviceset="PJ-" device="201"/>
-<part name="K2" library="con-subd" deviceset="M09HP" device=""/>
+<part name="J4" library="con-subd" deviceset="M09HP" device=""/>
 <part name="GND15" library="supply1" deviceset="GND" device=""/>
 <part name="T1(*)" library="transistor-npn" deviceset="BC338*" device=""/>
 <part name="K1(*)" library="relay" deviceset="351" device=""/>
+<part name="J12(*)" library="AudioJack" deviceset="PJ-325" device=""/>
 </parts>
 <sheets>
@@
 <text x="218.44" y="20.32" size="2.54" layer="94" font="vector">Danjovic 2021</text>
 <text x="163.83" y="16.002" size="5.08" layer="94" font="vector" ratio="14">CASIO FA-32</text>
-<wire x1="38.1" y1="20.32" x2="66.04" y2="20.32" width="0.1524" layer="97" style="shortdash"/>
+<wire x1="43.18" y1="17.78" x2="71.12" y2="17.78" width="0.1524" layer="97" style="shortdash"/>
 </plain>
 <instances>
@@
 <instance part="J2" gate="G$1" x="15.24" y="114.3"/>
 <instance part="J3" gate="G$1" x="15.24" y="55.88" rot="MR180"/>
-<instance part="K2" gate="G$1" x="215.9" y="91.44" rot="R90"/>
+<instance part="J4" gate="G$1" x="215.9" y="91.44" rot="R90"/>
 <instance part="GND15" gate="1" x="208.28" y="106.68" smashed="yes">
 <attribute name="VALUE" x="205.74" y="104.14" size="1.778" layer="96"/>
 </instance>
-<instance part="T1(*)" gate="G$1" x="93.98" y="20.32" smashed="yes" rot="MR0">
-<attribute name="NAME" x="88.9" y="20.32" size="1.778" layer="95" rot="MR0"/>
-<attribute name="VALUE" x="88.9" y="17.78" size="1.778" layer="96" rot="MR0"/>
-</instance>
-<instance part="K1(*)" gate="1" x="71.12" y="20.32"/>
-<instance part="K1(*)" gate="2" x="35.56" y="17.78"/>
-<instance part="K1(*)" gate="3" x="55.88" y="17.78"/>
+<instance part="T1(*)" gate="G$1" x="99.06" y="17.78" smashed="yes" rot="MR0">
+<attribute name="NAME" x="93.98" y="17.78" size="1.778" layer="95" rot="MR0"/>
+<attribute name="VALUE" x="93.98" y="15.24" size="1.778" layer="96" rot="MR0"/>
+</instance>
+<instance part="K1(*)" gate="1" x="76.2" y="17.78"/>
+<instance part="K1(*)" gate="2" x="40.64" y="15.24"/>
+<instance part="K1(*)" gate="3" x="60.96" y="15.24"/>
+<instance part="J12(*)" gate="G$1" x="15.24" y="20.32" rot="MR0"/>
 </instances>
 <busses>
@@
 <label x="27.94" y="137.16" size="1.778" layer="95"/>
 </segment>
+<segment>
+<wire x1="27.94" y1="22.86" x2="30.48" y2="22.86" width="0.1524" layer="91"/>
+<pinref part="J12(*)" gate="G$1" pin="5"/>
+</segment>
 </net>
 <net name="PE" class="0">
@@
 <segment>
 <pinref part="PE7" gate="M" pin="PE"/>
-<pinref part="K2" gate="G$1" pin="G1"/>
+<pinref part="J4" gate="G$1" pin="G1"/>
 <wire x1="208.28" y1="83.82" x2="208.28" y2="60.96" width="0.1524" layer="91"/>
-<pinref part="K2" gate="G$1" pin="G2"/>
+<pinref part="J4" gate="G$1" pin="G2"/>
 <wire x1="208.28" y1="60.96" x2="208.28" y2="58.42" width="0.1524" layer="91"/>
 <wire x1="223.52" y1="83.82" x2="223.52" y2="60.96" width="0.1524" layer="91"/>
@@
 <junction x="43.18" y="124.46"/>
 <pinref part="J2" gate="G$1" pin="R"/>
-<wire x1="22.86" y1="116.84" x2="35.56" y2="116.84" width="0.1524" layer="91"/>
+<wire x1="22.86" y1="116.84" x2="25.4" y2="116.84" width="0.1524" layer="91"/>
+<wire x1="25.4" y1="116.84" x2="35.56" y2="116.84" width="0.1524" layer="91"/>
 <wire x1="35.56" y1="116.84" x2="35.56" y2="124.46" width="0.1524" layer="91"/>
 <junction x="35.56" y="124.46"/>
 <pinref part="J1" gate="G$1" pin="R"/>
-<wire x1="22.86" y1="132.08" x2="35.56" y2="132.08" width="0.1524" layer="91"/>
+<wire x1="22.86" y1="132.08" x2="25.4" y2="132.08" width="0.1524" layer="91"/>
+<wire x1="25.4" y1="132.08" x2="35.56" y2="132.08" width="0.1524" layer="91"/>
 <wire x1="35.56" y1="132.08" x2="35.56" y2="124.46" width="0.1524" layer="91"/>
 <label x="27.94" y="116.84" size="1.778" layer="95"/>
 <label x="27.94" y="132.08" size="1.778" layer="95"/>
+<pinref part="J2" gate="G$1" pin="C"/>
+<wire x1="22.86" y1="114.3" x2="25.4" y2="114.3" width="0.1524" layer="91"/>
+<wire x1="25.4" y1="114.3" x2="25.4" y2="116.84" width="0.1524" layer="91"/>
+<junction x="25.4" y="116.84"/>
+<pinref part="J1" gate="G$1" pin="C"/>
+<wire x1="22.86" y1="134.62" x2="25.4" y2="134.62" width="0.1524" layer="91"/>
+<wire x1="25.4" y1="134.62" x2="25.4" y2="132.08" width="0.1524" layer="91"/>
+<junction x="25.4" y="132.08"/>
 </segment>
 <segment>
@@
 <label x="193.04" y="88.9" size="1.778" layer="95"/>
 <wire x1="170.18" y1="71.12" x2="215.9" y2="71.12" width="0.1524" layer="91"/>
-<pinref part="K2" gate="G$1" pin="8"/>
+<pinref part="J4" gate="G$1" pin="8"/>
 <wire x1="215.9" y1="83.82" x2="215.9" y2="71.12" width="0.1524" layer="91"/>
 </segment>
@@
 </segment>
 <segment>
-<pinref part="K2" gate="G$1" pin="3"/>
+<pinref part="J4" gate="G$1" pin="3"/>
 <wire x1="215.9" y1="99.06" x2="215.9" y2="111.76" width="0.1524" layer="91"/>
 <wire x1="215.9" y1="111.76" x2="208.28" y2="111.76" width="0.1524" layer="91"/>
@@
 </segment>
 <segment>
-<wire x1="91.44" y1="12.7" x2="91.44" y2="15.24" width="0.1524" layer="91"/>
+<wire x1="96.52" y1="10.16" x2="96.52" y2="12.7" width="0.1524" layer="91"/>
 <pinref part="T1(*)" gate="G$1" pin="E"/>
+</segment>
+<segment>
+<wire x1="27.94" y1="12.7" x2="30.48" y2="12.7" width="0.1524" layer="91"/>
+<pinref part="J12(*)" gate="G$1" pin="1"/>
+</segment>
+<segment>
+<wire x1="27.94" y1="17.78" x2="30.48" y2="17.78" width="0.1524" layer="91"/>
+<pinref part="J12(*)" gate="G$1" pin="2"/>
+</segment>
+<segment>
+<wire x1="27.94" y1="20.32" x2="30.48" y2="20.32" width="0.1524" layer="91"/>
+<pinref part="J12(*)" gate="G$1" pin="4"/>
 </segment>
 </net>
@@
 <label x="27.94" y="111.76" size="1.778" layer="95"/>
 </segment>
+<segment>
+<wire x1="30.48" y1="15.24" x2="27.94" y2="15.24" width="0.1524" layer="91"/>
+<pinref part="J12(*)" gate="G$1" pin="3"/>
+</segment>
 </net>
 <net name="REM-" class="0">
@@
 </segment>
 <segment>
-<wire x1="50.8" y1="22.86" x2="48.26" y2="22.86" width="0.1524" layer="91"/>
+<wire x1="55.88" y1="20.32" x2="53.34" y2="20.32" width="0.1524" layer="91"/>
 <pinref part="K1(*)" gate="3" pin="S"/>
 </segment>
@@
 </segment>
 <segment>
-<wire x1="55.88" y1="12.7" x2="55.88" y2="15.24" width="0.1524" layer="91"/>
+<wire x1="60.96" y1="10.16" x2="60.96" y2="12.7" width="0.1524" layer="91"/>
 <pinref part="K1(*)" gate="3" pin="P"/>
 </segment>
@@
 </segment>
 <segment>
-<wire x1="91.44" y1="27.94" x2="91.44" y2="25.4" width="0.1524" layer="91"/>
+<wire x1="96.52" y1="25.4" x2="96.52" y2="22.86" width="0.1524" layer="91"/>
 <pinref part="T1(*)" gate="G$1" pin="C"/>
 </segment>
 <segment>
-<wire x1="71.12" y1="15.24" x2="71.12" y2="12.7" width="0.1524" layer="91"/>
+<wire x1="76.2" y1="12.7" x2="76.2" y2="10.16" width="0.1524" layer="91"/>
 <pinref part="K1(*)" gate="1" pin="2"/>
 </segment>
@@
 <wire x1="220.98" y1="116.84" x2="220.98" y2="99.06" width="0.1524" layer="91"/>
 <label x="220.98" y="109.22" size="1.778" layer="95" rot="R90"/>
-<pinref part="K2" gate="G$1" pin="5"/>
+<pinref part="J4" gate="G$1" pin="5"/>
 </segment>
 <segment>
@@
 </segment>
 <segment>
-<wire x1="71.12" y1="25.4" x2="71.12" y2="27.94" width="0.1524" layer="91"/>
+<wire x1="76.2" y1="22.86" x2="76.2" y2="25.4" width="0.1524" layer="91"/>
 <pinref part="K1(*)" gate="1" pin="1"/>
 </segment>
@@
 <wire x1="241.3" y1="43.18" x2="241.3" y2="78.74" width="0.1524" layer="91"/>
 <label x="231.14" y="81.28" size="1.778" layer="95"/>
-<pinref part="K2" gate="G$1" pin="6"/>
+<pinref part="J4" gate="G$1" pin="6"/>
 <wire x1="210.82" y1="83.82" x2="210.82" y2="78.74" width="0.1524" layer="91"/>
 <wire x1="210.82" y1="78.74" x2="241.3" y2="78.74" width="0.1524" layer="91"/>
@@
 </segment>
 <segment>
-<wire x1="96.52" y1="20.32" x2="99.06" y2="20.32" width="0.1524" layer="91"/>
+<wire x1="101.6" y1="17.78" x2="104.14" y2="17.78" width="0.1524" layer="91"/>
 <pinref part="T1(*)" gate="G$1" pin="B"/>
 </segment>
@@
 <wire x1="203.2" y1="142.24" x2="243.84" y2="142.24" width="0.1524" layer="91"/>
 <label x="233.68" y="96.52" size="1.778" layer="95"/>
-<pinref part="K2" gate="G$1" pin="9"/>
+<pinref part="J4" gate="G$1" pin="9"/>
 <wire x1="218.44" y1="83.82" x2="218.44" y2="71.12" width="0.1524" layer="91"/>
 <wire x1="218.44" y1="71.12" x2="243.84" y2="71.12" width="0.1524" layer="91"/>
@@
 <junction x="132.08" y="101.6"/>
 <label x="193.04" y="101.6" size="1.778" layer="95"/>
-<pinref part="K2" gate="G$1" pin="1"/>
+<pinref part="J4" gate="G$1" pin="1"/>
 <wire x1="210.82" y1="101.6" x2="210.82" y2="99.06" width="0.1524" layer="91"/>
 </segment>

Commit message: Updated files
Other:
- moved on the sheet: C1, C10, C11, C12, C13, C14, C15, C16, C2, C3, C4, C5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
