File: Schematics/HOTBIT HB8000/HotBit.sch (EAGLE design)
At the start: 150 parts, among them IC1 4416, IC6 4416, J1 TOP SLOT, J10 CON_AV, J15 POWER, J2 SIDE SLOT, J20 IMPRESSORA, J25 TECLADO, J3 CASSETE, SW1 RESET, T1 BC550, T2 BC550, T3 BC550, T4 BC550, X1 10.726, X2 AUDIO OUT

Commit message: Added RF modulator, corrected main board schematic
Added rebuilt schematics of RF modulator, corrected supply voltage for RF modulator on main board (was 5V instead of 12V) and updated library with LM1889 modulator
Connections:
- net +12V: now also J10.VCC
- net +5V: no longer J10.VCC
Other:
- note added: "A"
- note added: "Rev A: Correcao Alimentacao Conector AV, Maio 2019"
- note removed: "-"
Changed lines of the file:
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@@
 <part name="J10" library="hotbit" deviceset="CON_AV" device=""/>
 <part name="J15" library="hotbit" deviceset="CON-PWR" device="" value="POWER"/>
-<part name="P+40" library="supply1" deviceset="+5V" device=""/>
 <part name="GND40" library="supply1" deviceset="GND" device=""/>
 <part name="P+41" library="supply1" deviceset="+12V" device=""/>
@@
 <part name="GND56" library="supply1" deviceset="GND" device=""/>
 <part name="P+49" library="supply1" deviceset="+5V" device=""/>
+<part name="P+50" library="supply1" deviceset="+12V" device=""/>
 </parts>
 <sheets>
@@
 <text x="349.25" y="-262.89" size="1.778" layer="94" font="vector" ratio="14">Redesenhado por Danjovic, Jan 2018</text>
 <text x="-391.16" y="-45.72" size="1.778" layer="94">Rev-: Desenho inicial, Jan 2018</text>
-<text x="441.96" y="-284.48" size="2.54" layer="94" font="vector" ratio="14">-</text>
+<text x="441.96" y="-284.48" size="2.54" layer="94" font="vector" ratio="14">A</text>
 <text x="349.25" y="-265.43" size="1.778" layer="94" font="vector" ratio="14">htp://hotbit.blogger.com     danjovic@hotmail.com   </text>
 <text x="247.904" y="25.4" size="2.54" layer="92" font="vector" ratio="13" rot="R90">ADDRESS BUS</text>
+<text x="-391.16" y="-48.26" size="1.778" layer="94">Rev A: Correcao Alimentacao Conector AV, Maio 2019</text>
 </plain>
 <instances>
@@
 <instance part="J10" gate="G$1" x="401.32" y="-7.62" rot="MR180"/>
 <instance part="J15" gate="G$1" x="-215.9" y="-63.5" rot="R180"/>
-<instance part="P+40" gate="1" x="393.7" y="7.62" smashed="yes">
-<attribute name="VALUE" x="396.24" y="7.62" size="1.778" layer="96" rot="R90"/>
-</instance>
 <instance part="GND40" gate="1" x="386.08" y="0"/>
 <instance part="P+41" gate="1" x="-195.58" y="-63.5" smashed="yes" rot="MR90">
@@
 <attribute name="VALUE" x="175.26" y="-144.78" size="1.778" layer="96" rot="R180"/>
 </instance>
+<instance part="P+50" gate="1" x="393.7" y="12.7" smashed="yes" rot="MR0">
+<attribute name="VALUE" x="395.224" y="16.51" size="1.778" layer="96" rot="MR180"/>
+</instance>
 </instances>
 <busses>
@@
 </segment>
 <segment>
-<pinref part="J10" gate="G$1" pin="VCC"/>
-<pinref part="P+40" gate="1" pin="+5V"/>
-<wire x1="393.7" y1="5.08" x2="393.7" y2="0" width="0.1524" layer="91"/>
-</segment>
-<segment>
 <pinref part="J15" gate="G$1" pin="+5V"/>
 <pinref part="P+42" gate="1" pin="+5V"/>
@@
 <pinref part="P+44" gate="1" pin="+12V"/>
 </segment>
+<segment>
+<pinref part="J10" gate="G$1" pin="VCC"/>
+<pinref part="P+50" gate="1" pin="+12V"/>
+<wire x1="393.7" y1="10.16" x2="393.7" y2="0" width="0.1524" layer="91"/>
+</segment>
 </net>

Commit message: fixed name of signals on printer port
Connections:
- removed net BSYRD: CI-13A.Y2, CI-2B.CLK
- new net !BSYRD: CI-11B1.G, CI-13A.Y4
- net !STBWR: now also CI-13A.Y2, CI-2B.CLK; no longer CI-11B1.G, CI-13A.Y4
Other:
- note added: "B"
- note added: "Rev B: Correcao nomes sinais porta Impressora, Marco 2025"
- note removed: "A"
Changed lines of the file:
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@@
 <?xml version="1.0" encoding="utf-8"?>
 <!DOCTYPE eagle SYSTEM "eagle.dtd">
-<eagle version="6.5.0">
+<eagle version="7.2.0">
 <drawing>
 <settings>
@@
 <text x="349.25" y="-262.89" size="1.778" layer="94" font="vector" ratio="14">Redesenhado por Danjovic, Jan 2018</text>
 <text x="-391.16" y="-45.72" size="1.778" layer="94">Rev-: Desenho inicial, Jan 2018</text>
-<text x="441.96" y="-284.48" size="2.54" layer="94" font="vector" ratio="14">A</text>
+<text x="441.96" y="-284.48" size="2.54" layer="94" font="vector" ratio="14">B</text>
 <text x="349.25" y="-265.43" size="1.778" layer="94" font="vector" ratio="14">htp://hotbit.blogger.com     danjovic@hotmail.com   </text>
 <text x="247.904" y="25.4" size="2.54" layer="92" font="vector" ratio="13" rot="R90">ADDRESS BUS</text>
 <text x="-391.16" y="-48.26" size="1.778" layer="94">Rev A: Correcao Alimentacao Conector AV, Maio 2019</text>
+<text x="-391.16" y="-50.8" size="1.778" layer="94">Rev B: Correcao nomes sinais porta Impressora, Marco 2025</text>
 </plain>
 <instances>
@@
 </segment>
 </net>
-<net name="BSYRD" class="0">
+<net name="!STBWR" class="0">
 <segment>
 <pinref part="CI-2" gate="B" pin="CLK"/>
@@
 </segment>
 </net>
-<net name="!STBWR" class="0">
+<net name="!BSYRD" class="0">
 <segment>
 <pinref part="CI-13" gate="A" pin="Y4"/>
